File: H18R11/Design/H18R11.brd (EAGLE design)
At the start: 60 x 34.6 mm, 19 parts, among them P2 HEXABIT_X2_P1_P5_EDIT_POWER_P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, U1 STM32G0B1CEU6N, X1 XTALL_CSTCE8M00G52

Commit message: - Initial schematic design.
Parts:
- added C10: 100nF, HEXABITZ_RCLS:C-0603
- added C11, C12: 470nF, HEXABITZ_RCLS:C-0603
- added C13: (no value), HEXABITZ_RCLS:C-0603-POL
- added C14, C15, C22: 1nF, HEXABITZ_RCLS:C-0603
- added C16, C17, C9: 1uF, HEXABITZ_RCLS:C-0603
- added C18, C19: (no value), HEXABITZ_RCLS:C-0603
- added C20, C21: 10nF, HEXABITZ_RCLS:C-0603
- added C8: 220nF, HEXABITZ_RCLS:C-0603
- added D2, D3, D4, D5: Yellow, Hexabitz:VLMS1300-GS08
- added IC1: STSPIN948, HEXABITZ_ICs:QFN50P700X700X105-49N
- added P1, P3: (no value), HEXABITZ_CONNECTION_PARTS:1546111-2
- added R10, R9: 100R, HEXABITZ_RCLS:R-0603
- added R11, R12: (no value), HEXABITZ_RCLS:R-0603
- added R13, R14: 39k, HEXABITZ_RCLS:R-0603
- added R15: 18k, HEXABITZ_RCLS:R-0603
- added R16, R17, R18, R19: 10k, HEXABITZ_RCLS:R-0805
- added R4, R5: 50m, HEXABITZ_RCLS:R2512
- added R6: 5.6k, HEXABITZ_RCLS:R-0603
- added R7, R8: 22k, HEXABITZ_RCLS:R-0603
Connections:
- new net EN/FAULTA: C20.1, IC1.19, R14.1
- new net EN/FAULTB: C21.1, IC1.20, R13.1
- new net N$10: IC1.1, IC1.10, IC1.2, IC1.3, IC1.4, R4.2
- new net N$11: IC1.27, IC1.33, IC1.34, IC1.35, IC1.36, R5.2
- new net N$12: IC1.31, R6.2
- new net N$13: C14.1, IC1.23, R7.2
- new net N$14: IC1.11, R9.2
- new net N$15: IC1.26, R10.1
- new net N$16: C15.1, IC1.24, R8.2
- new net N$17: C19.1, IC1.21, R12.2
- new net N$18: C18.1, IC1.22, R11.1
- new net N$19: D3.C, R18.2
- new net N$21: D5.C, R16.2
- new net N$22: D4.C, R17.2
- new net N$23: D2.C, R19.2
- new net N$3: C9.1, IC1.6
- new net N$4: C9.2, IC1.9
- new net N$7: C10.1, IC1.7
- new net N$9: C10.2, IC1.8
- new net NSTBY: C22.1, IC1.13, R15.1
- new net OUT1A: D2.A, IC1.45, IC1.46, P1.2
- new net OUT1B: D4.A, D5.A, IC1.39, IC1.40, P3.2
- new net OUT2A: D3.A, IC1.47, IC1.48, P1.1
- new net OUT2B: IC1.37, IC1.38, P3.1
- new net PHA: IC1.15
- new net PHB: IC1.17
- new net PWM1A: IC1.14
- new net PWM1B: IC1.16
- new net REFA: R12.1
- new net REFB: R11.2
- new net VA: C16.1, R9.1
- new net VB: C17.1, R10.2
- net GND: now also C11.2, C12.2, C13.2, C14.2, C15.2, C16.2, C17.2, C18.2, C19.2, C20.2, C21.2, C22.2, C8.2, IC1.12, IC1.25, IC1.28, IC1.30, IC1.32, IC1.5, R16.1, R17.1, R18.1, R19.1, R4.1, R5.1, R6.1, R7.1, R8.1
- net VDD: now also C11.1, C12.1, C13.1, C8.1, IC1.18, IC1.29, IC1.41, IC1.42, IC1.43, IC1.44, R13.2, R14.2, R15.2

Commit message: - New schematic design - Initial Layout setup - Generated documentation
Parts:
- removed D16: BOURNS_CDSOD323-T03SCBOURNS_CDSOD323-T03SC_0_0, HEXABITZ_RCLS:BOURNS_CDSOD323-T03SC_0
- removed IC1: STSPIN948, HEXABITZ_ICs:QFN50P700X700X105-49N
- added Q1: TL431QDBZR,215, HEXABITZ_RCLS:SOT23_TO-236AB_NEX
- added R20, R21: 50m, HEXABITZ_RCLS:R2512
- added R22, R23, R24, R25, R26, R27, R28, R29, R30, R31, R32, R33, R34, R35, R36, R37, R38, R39, R40, R41, R42: (no value), HEXABITZ_RCLS:R-0402
- added U$1: HEXABIT_17.32_X3_NO_P1_P2_P3_P4_P5_P6_P11_P12, hexabitz_connectors:HEXABIT_17.32_X3_NO_P1_P2_P3_P4_P5_P6_P11_P12
- added U2: TSV772IQ2T_SEPARATED_SYMBOLSSON50P200X200X60-9N, HEXABITZ_ICs:SON50P200X200X60-9N
- added U3: STSPIN948, HEXABITZ_ICs:QFN50P700X700X105-49N
- C13: value (none) -> 100nF; device HEXABITZ_RCLS:C-0603-POL -> HEXABITZ_RCLS:C-0603
- C5: value 100nF -> 220uF; device HEXABITZ_RCLS:C-0603 -> HEXABITZ_RCLS:CAPPRD500W60D1250H2500
- C7: value 4.7uF -> 220uF; device HEXABITZ_RCLS:C-0805-POL -> HEXABITZ_RCLS:CAPPRD500W60D1250H2500
- P2: value HEXABIT_X2_P1_P5_EDIT_POWER_PADS -> (none); device hexabitz_connectors:HEXABIT_X2_P1_P5_EDIT_POWER_PADS -> HEXABITZ_CONNECTION_PARTS:1546111-2
- moved R19 229.4 mm to (19.1, -14.6), turned to 30 degrees
- moved R18 222.3 mm to (15.1, -16.8), turned to 30 degrees
- moved R17 215.9 mm to (-18.4, -14.9), turned to 150 degrees
- moved R15 212.4 mm to (4.60, 16.8), turned to 90 degrees
- moved R16 209.3 mm to (-13.5, -17.8), turned to 330 degrees
- moved D5 201.1 mm to (-14.1, -19.4), turned to 60 degrees
- moved D4 197.6 mm to (-19.5, -16.2), turned to 240 degrees
- moved D3 194.2 mm to (16.0, -18.3), turned to 120 degrees
- moved D2 191.4 mm to (20.3, -15.9), turned to 120 degrees
- moved R5 168.2 mm to (-10.0, -2.06), turned to 90 degrees
- moved R4 155.9 mm to (12.4, -2.22), turned to 90 degrees
- moved C22 150.5 mm to (3.65, 19.8), turned to 90 degrees
- moved C21 142.6 mm to (-0.48, 21.7), turned to 90 degrees
- moved C20 140.0 mm to (1.59, 21.7), turned to 90 degrees
- moved R12 134.1 mm to (-2.54, 26.2), turned to 90 degrees
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Connections:
- removed net OUT1A: D2.A, IC1.45, IC1.46, P1.2
- removed net OUT1B: D4.A, D5.A, IC1.39, IC1.40, P3.2
- new net +VS: C11.1, C12.1, C13.1, C5.P, C7.P, P2.1, U3.41, U3.42, U3.43, U3.44
- new net ACS+: R20.2, R27.2, U3.45, U3.46
- new net ACS-: D2.A, P3.2, R20.1, R26.2
- new net BCS+: R21.2, R34.2, U3.39, U3.40
- new net BCS-: D4.A, P1.1, R21.1, R33.2
- new net N$20: R25.2, U2.1
- new net N$24: R24.2, R25.1, U2.2
- new net N$25: R31.2, R41.1, R42.1
- new net N$26: R24.1, R26.1, R29.2
- new net N$27: R22.1, R27.1, R28.2
- new net N$28: R37.2, U2.7
- new net N$29: R32.2, R37.1, U2.6
- new net N$31: R32.1, R33.1, R36.2
- new net N$32: R30.1, R34.1, R35.2
- new net N$33: R22.2, R23.1, U2.3
- new net N$34: R23.2, R39.1, R40.1
- new net VREF: Q1.1, Q1.2, R30.2, R31.1, R38.1, R39.2, R41.2, U2.5
- net EN/FAULTA: now also U3.19; no longer IC1.19
- net EN/FAULTB: now also U3.20; no longer IC1.20
- net GND: now also Q1.3, R28.1, R29.1, R35.1, R36.1, R40.2, R42.2, U$1.PAD_PD12, U$1.PAD_PD17, U$1.PAD_PD19, U2.4, U2.9, U3.12, U3.25, U3.28, U3.30, U3.32, U3.5; no longer C11.2, C12.2, C13.2, C5.2, C7.2, IC1.12, IC1.25, IC1.28, IC1.30, IC1.32, IC1.5, P2.PAD_PD11, P2.PAD_PD12, P2.PAD_PD13, P2.PAD_PD14, P2.PAD_PD17, P2.PAD_PD18, P2.PAD_PD19, P2.PAD_PD20
- net N$10: now also U3.1, U3.10, U3.2, U3.3, U3.4; no longer IC1.1, IC1.10, IC1.2, IC1.3, IC1.4
- net N$11: now also U3.27, U3.33, U3.34, U3.35, U3.36; no longer IC1.27, IC1.33, IC1.34, IC1.35, IC1.36
- net N$12: now also U3.31; no longer IC1.31
- net N$13: now also U3.23; no longer IC1.23
- net N$14: now also U3.11; no longer IC1.11
- net N$15: now also U3.26; no longer IC1.26
- net N$16: now also U3.24; no longer IC1.24
- net N$17: now also U3.21; no longer IC1.21
- net N$18: now also U3.22; no longer IC1.22
- net N$3: now also U3.6; no longer IC1.6
- net N$4: now also U3.9; no longer IC1.9
- net N$7: now also U3.7; no longer IC1.7
- net N$9: now also U3.8; no longer IC1.8
- net NSTBY: now also U3.13; no longer IC1.13
- net OUT2A: now also P3.1, U3.47, U3.48; no longer IC1.47, IC1.48, P1.1
- net OUT2B: now also D5.A, P1.2, U3.37, U3.38; no longer IC1.37, IC1.38, P3.1
- net PHA: now also U3.15; no longer IC1.15
- net PHB: now also U3.17; no longer IC1.17
- net PWM1A: now also U3.14; no longer IC1.14
- net PWM1B: now also U3.16; no longer IC1.16
- net USART1_RX: now also U$1.PAD_PD8; no longer P2.PAD_PD4
- net USART1_TX: now also U$1.PAD_PU8; no longer P2.PAD_PU4
- net USART2_RX: now also U$1.PAD_PD1; no longer P2.PAD_PD2
- net USART2_TX: now also U$1.PAD_PU1; no longer P2.PAD_PU2
- net USART3_RX: now also U$1.PAD_PD2; no longer P2.PAD_PD3
- net USART3_TX: now also U$1.PAD_PU2; no longer P2.PAD_PU3
- net USART5_RX: no longer P2.PAD_PD5
- net USART5_TX: no longer P2.PAD_PU5
- net USART6_RX: now also U$1.PAD_PD3; no longer P2.PAD_PD1
- net USART6_TX: now also U$1.PAD_PU3; no longer P2.PAD_PU1
- net VDD: now also R38.2, U$1.PAD_PU12, U$1.PAD_PU17, U$1.PAD_PU19, U2.8, U3.18, U3.29; no longer C11.1, C12.1, C13.1, C5.1, C7.1, IC1.18, IC1.29, IC1.41, IC1.42, IC1.43, IC1.44, P2.PAD_PU11, P2.PAD_PU12, P2.PAD_PU13, P2.PAD_PU14, P2.PAD_PU17, P2.PAD_PU18, P2.PAD_PU19, P2.PAD_PU20
- net VDDA: no longer D16.2
- net VSSA: now also C11.2, C12.2, C13.2, C5.N, C7.N, P2.2; no longer D16.1
Routing:
- net USART2_TX: track 18.1 -> 0.00 mm, vias 1 -> 0
- net USART6_TX: track 17.7 -> 0.00 mm, vias 1 -> 0
- net USART1_TX: track 16.9 -> 0.00 mm, vias 1 -> 0
- net USART3_TX: track 15.2 -> 0.00 mm, vias 1 -> 0
- net USART6_RX: track 14.9 -> 0.00 mm
- net USART5_RX: track 14.5 -> 0.00 mm
- net USART5_TX: track 14.3 -> 0.00 mm, vias 1 -> 0
- net USART2_RX: track 14.2 -> 0.00 mm
- net N$8: track 12.4 -> 0.00 mm
- net USART1_RX: track 12.1 -> 0.00 mm
- net USART3_RX: track 10.8 -> 0.00 mm
- net CLK: track 9.53 -> 0.00 mm
- net DATA: track 8.29 -> 0.00 mm
- net VDDA: track 7.72 -> 0.00 mm, vias 1 -> 0
- net GND: track 6.49 -> 0.00 mm
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Other:
- board size 60 x 34.6 mm -> 60 x 60.6 mm
- board text removed: "P5"
