File: H18R11/Design/H18R11.sch (EAGLE design)
At the start: 19 parts, among them P2 HEXABIT_X2_P1_P5_EDIT_POWER_P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, U1 STM32G0B1CEU6N, X1 XTALL_CSTCE8M00G52

Commit message: - Initial schematic design.
Parts:
- added C10: 100nF, HEXABITZ_RCLS:C-0603
- added C11, C12: 470nF, HEXABITZ_RCLS:C-0603
- added C13: C-0603-POL, HEXABITZ_RCLS:C-0603-POL
- added C14, C15, C22: 1nF, HEXABITZ_RCLS:C-0603
- added C16, C17, C9: 1uF, HEXABITZ_RCLS:C-0603
- added C18, C19: (no value), HEXABITZ_RCLS:C-0603
- added C20, C21: 10nF, HEXABITZ_RCLS:C-0603
- added C8: 220nF, HEXABITZ_RCLS:C-0603
- added D2, D3, D4, D5: Yellow, Hexabitz:VLMS1300-GS08
- added IC1: STSPIN948, HEXABITZ_ICs:STSPIN948
- added P1, P3: (no value), HEXABITZ_CONNECTION_PARTS:1546111-2
- added R10, R9: 100R, HEXABITZ_RCLS:R-0603
- added R11, R12: (no value), HEXABITZ_RCLS:R-0603
- added R13, R14: 39k, HEXABITZ_RCLS:R-0603
- added R15: 18k, HEXABITZ_RCLS:R-0603
- added R16, R17, R18, R19: 10k, HEXABITZ_RCLS:R-0805
- added R4, R5: 50m, HEXABITZ_RCLS:R-US_R2512
- added R6: 5.6k, HEXABITZ_RCLS:R-0603
- added R7, R8: 22k, HEXABITZ_RCLS:R-0603
Connections:
- new net EN/FAULTA: C20.1, IC1.EN/NFAULTA, R14.1
- new net EN/FAULTB: C21.1, IC1.EN/NFAULTB, R13.1
- new net N$10: IC1.LSS1A_1, IC1.LSS1A_2, IC1.LSS2A_1, IC1.LSS2A_2, IC1.SENSEA, R4.2
- new net N$11: IC1.LSS1B_1, IC1.LSS1B_2, IC1.LSS2B_1, IC1.LSS2B_2, IC1.SENSEB, R5.2
- new net N$12: IC1.SR, R6.2
- new net N$13: C14.1, IC1.TOFFA, R7.2
- new net N$14: IC1.VA, R9.2
- new net N$15: IC1.VB, R10.1
- new net N$16: C15.1, IC1.TOFFB, R8.2
- new net N$17: C19.1, IC1.REFA, R12.2
- new net N$18: C18.1, IC1.REFB, R11.1
- new net N$19: D3.C, R18.2
- new net N$21: D5.C, R16.2
- new net N$22: D4.C, R17.2
- new net N$23: D2.C, R19.2
- new net N$3: C9.1, IC1.VSPUMP
- new net N$4: C9.2, IC1.VBOOT
- new net N$7: C10.1, IC1.CP1
- new net N$9: C10.2, IC1.CP2
- new net NSTBY: C22.1, IC1.NSTBY, R15.1
- new net OUT1A: D2.A, IC1.OUT1A_1, IC1.OUT1A_2, P1.2
- new net OUT1B: D4.A, D5.A, IC1.OUT1B_1, IC1.OUT1B_2, P3.2
- new net OUT2A: D3.A, IC1.OUT2A_1, IC1.OUT2A_2, P1.1
- new net OUT2B: IC1.OUT2B_1, IC1.OUT2B_2, P3.1
- new net PHA: IC1.PHA
- new net PHB: IC1.PHB
- new net PWM1A: IC1.PWM1A
- new net PWM1B: IC1.PWM1B
- new net REFA: R12.1
- new net REFB: R11.2
- new net VA: C16.1, R9.1
- new net VB: C17.1, R10.2
- net GND: now also C11.2, C12.2, C13.2, C14.2, C15.2, C16.2, C17.2, C18.2, C19.2, C20.2, C21.2, C22.2, C8.2, IC1.GND_1, IC1.GND_2, IC1.MODE1, IC1.MODE3, IC1.OFFSETA, IC1.OFFSETB, R16.1, R17.1, R18.1, R19.1, R4.1, R5.1, R6.1, R7.1, R8.1
- net VDD: now also C11.1, C12.1, C13.1, C8.1, IC1.MODE2, IC1.VDD, IC1.VS_1, IC1.VS_2, IC1.VS_3, IC1.VS_4, R13.2, R14.2, R15.2

Commit message: - New schematic design - Initial Layout setup - Generated documentation
Parts:
- removed D16: BOURNS_CDSOD323-T03SCBOURNS_CDSOD323-T03SC_0_0, HEXABITZ_RCLS:BOURNS_CDSOD323-T03SCBOURNS_CDSOD323-T03SC_0_0
- added Q1: TL431QDBZR,215, HEXABITZ_RCLS:TL431QDBZR,215
- added R20, R21: 50m, HEXABITZ_RCLS:R-US_R2512
- added R22, R23, R24, R25, R26, R27, R28, R29, R30, R31, R32, R33, R34, R35, R36, R37, R38, R39, R40, R41, R42: (no value), HEXABITZ_RCLS:R-0402
- added U$1: HEXABIT_17.32_X3_NO_P1_P2_P3_P4_P5_P6_P11_P12, hexabitz_connectors:HEXABIT_17.32_X3_NO_P1_P2_P3_P4_P5_P6_P11_P12
- added U2: TSV772IQ2T_SEPARATED_SYMBOLSSON50P200X200X60-9N, HEXABITZ_ICs:TSV772IQ2T_SEPARATED_SYMBOLSSON50P200X200X60-9N
- C13: value C-0603-POL -> 100nF; device HEXABITZ_RCLS:C-0603-POL -> HEXABITZ_RCLS:C-0603; VOLTAGE_RATING (none) -> 100v
- C5: value 100nF -> 220uF; device HEXABITZ_RCLS:C-0603 -> HEXABITZ_RCLS:EEUFS2A221B; VOLT (none) -> 100v
- C7: value 4.7uF -> 220uF; device HEXABITZ_RCLS:C-0805-POL -> HEXABITZ_RCLS:EEUFS2A221B; VOLT (none) -> 100v
- P2: value HEXABIT_X2_P1_P5_EDIT_POWER_PADS -> (none); device hexabitz_connectors:HEXABIT_X2_P1_P5_EDIT_POWER_PADS -> HEXABITZ_CONNECTION_PARTS:1546111-2
- renumbered IC1 to U3
Connections:
- removed net OUT1A: D2.A, P1.2, U3.OUT1A_1, U3.OUT1A_2
- removed net OUT1B: D4.A, D5.A, P3.2, U3.OUT1B_1, U3.OUT1B_2
- new net +VS: C11.1, C12.1, C13.1, C5.P, C7.P, P2.1, U3.VS_1, U3.VS_2, U3.VS_3, U3.VS_4
- new net ACS+: R20.2, R27.2, U3.OUT1A_1, U3.OUT1A_2
- new net ACS-: D2.A, P3.2, R20.1, R26.2
- new net BCS+: R21.2, R34.2, U3.OUT1B_1, U3.OUT1B_2
- new net BCS-: D4.A, P1.1, R21.1, R33.2
- new net N$20: R25.2, U2(1).OUT
- new net N$24: R24.2, R25.1, U2(1).-IN
- new net N$25: R31.2, R41.1, R42.1
- new net N$26: R24.1, R26.1, R29.2
- new net N$27: R22.1, R27.1, R28.2
- new net N$28: R37.2, U2(2).OUT
- new net N$29: R32.2, R37.1, U2(2).-IN
- new net N$31: R32.1, R33.1, R36.2
- new net N$32: R30.1, R34.1, R35.2
- new net N$33: R22.2, R23.1, U2(1).+IN
- new net N$34: R23.2, R39.1, R40.1
- new net VREF: Q1.1, Q1.2, R30.2, R31.1, R38.1, R39.2, R41.2, U2(2).+IN
- net GND: now also Q1.3, R28.1, R29.1, R35.1, R36.1, R40.2, R42.2, U$1.GND1, U$1.GND2, U$1.GND3, U2P.V-; no longer C11.2, C12.2, C13.2, C5.2, C7.-, P2.GND1, P2.GND2, P2.GND3, P2.GND4, P2.GND5, P2.GND6, P2.GND7, P2.GND8
- net OUT2A: now also P3.1; no longer P1.1
- net OUT2B: now also D5.A, P1.2; no longer P3.1
- net USART1_RX: now also U$1.SD4; no longer P2.SD4
- net USART1_TX: now also U$1.SU4; no longer P2.SU4
- net USART2_RX: now also U$1.SD2; no longer P2.SD2
- net USART2_TX: now also U$1.SU2; no longer P2.SU2
- net USART3_RX: now also U$1.SD3; no longer P2.SD3
- net USART3_TX: now also U$1.SU3; no longer P2.SU3
- net USART5_RX: no longer P2.SD5
- net USART5_TX: no longer P2.SU5
- net USART6_RX: now also U$1.SD1; no longer P2.SD1
- net USART6_TX: now also U$1.SU1; no longer P2.SU1
- net VDD: now also R38.2, U$1.VDD1, U$1.VDD2, U$1.VDD3, U2P.V+; no longer C11.1, C12.1, C13.1, C5.1, C7.+, P2.VDD1, P2.VDD2, P2.VDD3, P2.VDD4, P2.VDD5, P2.VDD6, P2.VDD7, P2.VDD8, U3.VS_1, U3.VS_2, U3.VS_3, U3.VS_4
- net VDDA: no longer D16.C
- net VSSA: now also C11.2, C12.2, C13.2, C5.N, C7.N, P2.2; no longer D16.A
Other:
- note added: "3"
